File: bipolar_linear_supply/bipolar_linear_supply.kicad_pcb (KiCad board)
At the start: 2 copper layers, 92 x 52 mm, 27 parts, among them J2 3.5mm, J3 3.5mm, SW1 SW_SPST, T1 48 VAC CT, U1 LM317_TO-220, U2 LM337_TO220

Commit message: Add files via upload
Parts:
- added G***: LOGO, Fr_Logo:Fr1, F.Cu at (181.2, 96.8)
- added REF**: KiCad-Logo2_5mm_SilkScreen, Symbol:KiCad-Logo2_5mm_SilkScreen, F.Cu at (127.0, 62.2)
